Commit message: robot moves,but not correctly

File: tennis-description/urdf/laser.xacro (robot description, xacro)
@@ -36,5 +36,5 @@
               <!-- The URG-04LX-UG01  has  683 steps with 0.35139 Degree resolution -->
               <samples>720</samples>
-              <resolution>1</resolution>
+              <resolution>0.5</resolution>
               <max_angle>3.14</max_angle> <!-- 120 Degree -->
               <min_angle>-3.14</min_angle> <!-- -120 Degree -->
@@ -48,5 +48,5 @@
         </ray>
         <plugin name="laser" filename="libgazebo_ros_laser.so">
-          <robotNamespace></robotNamespace>
+          <robotNamespace>/leo</robotNamespace>
           <topicName>${name}/scan</topicName>
           <frameName>${name}</frameName>

File: tennis-description/urdf/leo.gazebo.xacro (robot description, xacro)
@@ -1,23 +1,25 @@
 <?xml version="1.0"?>
 <robot xmlns:xacro="http://www.ros.org/wiki/xacro" name="leo">
-  <gazebo>
-    <plugin name="differential_drive_controller" filename="libgazebo_ros_diff_drive.so">
-      <updateRate>100</updateRate>
-      <leftJoint>left_front_wheel_joint</leftJoint>
-      <rightJoint>right_front_wheel_joint</rightJoint>
-      <wheelSeparation>0.33</wheelSeparation>
-      <wheelDiameter>0.3</wheelDiameter>
-      <wheelAcceleration>false</wheelAcceleration>
-      <wheelTorque>50</wheelTorque>
-      <commandTopic>diff/cmd_vel</commandTopic>
-      <odometryTopic>diff/odom</odometryTopic>
-      <odometryFrame>odom</odometryFrame>
-      <robotBaseFrame>base_root</robotBaseFrame>
-      <odometrySource>1</odometrySource>
-      <publishWheelTF>false</publishWheelTF>
-      <publishOdomTF>true</publishOdomTF>
-      <publishWheelJointState>true</publishWheelJointState>
-    </plugin>
-  </gazebo>
+  <!-- <gazebo> -->
+  <!--   <plugin name="skid_steer" filename="libgazebo_ros_skid_steer_drive.so"> -->
+  <!--     <updateRate>100</updateRate> -->
+  <!--     <leftFrontJoint>left_front_wheel_joint</leftFrontJoint> -->
+  <!--     <leftRearJoint>left_back_wheel_joint</leftRearJoint> -->
+  <!--     <rightFrontJoint>right_front_wheel_joint</rightFrontJoint> -->
+  <!--     <rightRearJoint>right_back_wheel_joint</rightRearJoint> -->
+  <!--     <wheelSeparation>0.33</wheelSeparation> -->
+  <!--     <wheelDiameter>0.3</wheelDiameter> -->
+  <!--     <wheelAcceleration>false</wheelAcceleration> -->
+  <!--     <torque>100</torque> -->
+  <!--     <commandTopic>diff/cmd_vel</commandTopic> -->
+  <!--     <odometryTopic>diff/odom</odometryTopic> -->
+  <!--     <odometryFrame>odom</odometryFrame> -->
+  <!--     <robotBaseFrame>base_root</robotBaseFrame> -->
+  <!--     <odometrySource>1</odometrySource> -->
+  <!--     <publishWheelTF>false</publishWheelTF> -->
+  <!--     <publishOdomTF>true</publishOdomTF> -->
+  <!--     <publishWheelJointState>true</publishWheelJointState> -->
+  <!--   </plugin> -->
+  <!-- </gazebo> -->
   <gazebo reference="base">
     <material>Gazebo/Blue</material>
@@ -31,4 +33,5 @@
       <topic>imu</topic>
       <plugin filename="libgazebo_ros_imu_sensor.so" name="imu_plugin">
+        <robotNamespace>/leo</robotNamespace>
         <topicName>imu</topicName>
         <bodyName>imu_link</bodyName>
@@ -52,5 +55,5 @@
   <gazebo>
     <plugin name="gazebo_ros_control" filename="libgazebo_ros_control.so">
-      <robotNamespace>leo</robotNamespace>
+      <robotNamespace>/leo</robotNamespace>
     </plugin>
   </gazebo>

File: tennis-description/urdf/leo.xacro (robot description, xacro)
@@ -23,5 +23,5 @@
     </collision>
     <inertial>
-      <mass value="36" />
+      <mass value="30" />
       <inertia ixx="${robotlxx}" ixy="${robotlxy}" ixz="${robotlxz}" iyy="${robotlyy}" iyz="${robotlyz}" izz="${robotlzz}" />
     </inertial>
@@ -43,9 +43,19 @@
       </collision>
       <inertial>
-        <origin xyz="0 0 0" rpy="${pi/2} 0 0" />
+        <!-- <origin xyz="0 0 0" rpy="${pi/2} 0 0" /> -->
+        <origin xyz="0 0 0" rpy="0 0 0" />
         <mass value="1" />
-        <xacro:cylinder_inertia m="1" r="0.15" h="0.05" />
+        <xacro:cylinder_inertia m="3" r="0.15" h="0.05" />
       </inertial>
     </link>
+    <gazebo reference="${side}_wheel_link">
+      <!-- <material>Gazebo/DarkGrey</mate10ial> -->
+      <selfCollide>false</selfCollide>
+      <mu value="0.9" />
+      <mu2 value="0.9" />
+      <kp value="10000000.0" />
+      <kd value="1" />
+      <!-- <fdir1 value="1 0 0" /> -->
+    </gazebo>
     <joint name="${side}_wheel_joint" type="continuous">
       <parent link="base" />
@@ -53,5 +63,5 @@
       <origin xyz="${reflect_x * 0.25} ${reflect_y * 0.25} 0" rpy="1.570796 0 0" />
       <axis xyz="0 0 1" />
-      <!-- <dynamics damping="0.8" friction="2.0" /> -->
+      <dynamics damping="0.8" friction="100.0" />
     </joint>
     <xacro:wheel_gazebo prefix="${side}" />
@@ -79,5 +89,5 @@
   </link>
   <!-- Connect that link to the base link in the middle of the robot -->
-  <joint name="base_link_joint" type="fixed">
+  <joint name="base_root_joint" type="fixed">
     <origin xyz="0 0 0.15" rpy="0 0 0" />
     <parent link="base_root" />
