Commit message: got ekf working, something wrong with the transform from the lidar to the base of the robot. Walls appear on wrong side of the robot

File: tennis-description/urdf/rplidar.xacro (robot description, xacro)
@@ -5,4 +5,5 @@
   <xacro:property name="rplidar_mass" value="0.190" />
   <xacro:property name="rplidar_geometry">
+    <origin xyz="0 0 0" rpy="0 0 0 " />
     <geometry>
       <cylinder radius="${rplidar_r}" length="${rplidar_h}" />
@@ -18,4 +19,5 @@
       </collision>
       <inertial>
+        <origin xyz="0 0 0" rpy="0 0 0" />
         <xacro:cylinder_inertia m="${rplidar_mass}" r="${rplidar_r}" h="${rplidar_h}" />
         <mass value="${rplidar_mass}" />
@@ -23,4 +25,5 @@
     </link>
     <joint name="${name}_joint" type="fixed">
+      <!-- <axis xyz="0 0 1" /> -->
       <origin xyz="${xyz}" rpy="${rpy}" />
       <parent link="${parent}" />
@@ -32,4 +35,5 @@
         <visualize>false</visualize>
         <update_rate>10</update_rate>
+        <always_on>true</always_on>
         <ray>
           <scan>
