Commit message: Updated wheel and base origins

File: tennis-description/urdf/leo.xacro (robot description, xacro)
@@ -5,5 +5,5 @@
   <link name="base">
     <visual>
-      <origin xyz="0.5 0.166 0.125" rpy="0.0 0.0 0.0" />
+      <origin xyz="0.0 0.0 0.0" rpy="0.0 0.0 0.0" />
       <geometry>
         <box size="1 0.33 0.25" />
@@ -11,5 +11,5 @@
     </visual>
     <collision>
-      <origin xyz="0.5 0.166 0.125" rpy="0.0 0.0 0.0" />
+      <origin xyz="0.0 0.0 0.0" rpy="0.0 0.0 0.0" />
       <geometry>
         <box size="1 0.33 0.25" />
@@ -37,5 +37,5 @@
       <parent link="base" />
       <child link="wheel_${side}" />
-      <origin xyz="${reflect_x * 0.5} ${reflect_y * 0.5} 0" rpy="1.570796 0 0" />
+      <origin xyz="${reflect_x * 0.25} ${reflect_y * 0.25} 0" rpy="1.570796 0 0" />
       <axis xyz="0 0 1" />
     </joint>

Commit message: Changed lidar offsets

File: tennis-description/urdf/leo.xacro (robot description, xacro)
@@ -77,8 +77,4 @@
   </joint>
   <xacro:include filename="$(find gazebo_plugins)/test/multi_robot_scenario/xacro/laser/hokuyo.xacro" />
-  <xacro:laser name="laser_vert_bottom" parent="base" xyz="0.3157984464801903 -0.002068548615034871 0.5099999434059285" rpy="3.1354753 -1.3045001 0.0024658" meshes="package://gazebo_plugins/test/multi_robot_scenario/meshes/laser" />
-  <xacro:include filename="$(find velodyne_description)/urdf/VLP-16.urdf.xacro" />
-  <xacro:VLP-16 parent="base" name="laser_horiz" topic="laser_horiz/packets" hz="10" samples="440" gpu="false">
-    <origin xyz="0.2325416305773505 -0.0001380069427607134 1.920122926231907" rpy="-0.0012068 0.114646 -0.0015308" />
-  </xacro:VLP-16>
+  <xacro:laser name="laser_vert_bottom" parent="base" xyz="0.3157984464801903 -0.002068548615034871 0.25" rpy="3.14159 0.0 0.0" meshes="package://gazebo_plugins/test/multi_robot_scenario/meshes/laser" />
 </robot>

Commit message: robot moves, not correctly yet

File: tennis-description/urdf/leo.xacro (robot description, xacro)
@@ -71,10 +71,10 @@
     <origin xyz="0.0 0.0 0" rpy="0 0 0" />
   </joint>
-  <link name="odom" />
-  <joint name="odom_joint" type="fixed">
-    <parent link="base" />
-    <child link="odom" />
-    <origin xyz="0 0 0 " rpy="0 0 0" />
-  </joint>
+  <!-- <link name="odom" /> -->
+  <!-- <joint name="odom_joint" type="fixed"> -->
+  <!--   <parent link="odom" /> -->
+  <!--   <child link="base_root" /> -->
+  <!--   <origin xyz="0 0 0 " rpy="0 0 0" /> -->
+  <!-- </joint> -->
   <!-- Create a root link with no inertia to make the solver happy and raise the robot above the floor -->
   <link name="base_root">

Commit message: maps correctly now, moves weird

File: tennis-description/urdf/leo.xacro (robot description, xacro)
@@ -47,6 +47,6 @@
         <!-- <origin xyz="0 0 0" rpy="${pi/2} 0 0" /> -->
         <origin xyz="0 0 0" rpy="0 0 0" />
-        <mass value="1" />
-        <xacro:cylinder_inertia m="3" r="0.15" h="0.05" />
+        <mass value="2" />
+        <xacro:cylinder_inertia m="2" r="0.15" h="0.05" />
       </inertial>
     </link>
@@ -55,5 +55,5 @@
       <child link="${side}_wheel_link" />
       <origin xyz="${reflect_x * 0.25} ${reflect_y * 0.25} 0" rpy="1.570796 0 0" />
-      <axis xyz="0 0 1" />
+      <axis xyz="0 0 -1" />
       <dynamics damping="0.8" friction="100.0" />
     </joint>

Commit message: it works! navigation is working

File: tennis-description/urdf/leo.xacro (robot description, xacro)
@@ -35,4 +35,5 @@
     <link name="${side}_wheel_link">
       <visual>
+        <origin xyz=" 0 0 0" rpy="${pi/2} 0 0" />
         <geometry>
           <cylinder radius="0.15" length="0.05" />
@@ -40,4 +41,5 @@
       </visual>
       <collision>
+        <origin xyz=" 0 0 0" rpy="${pi/2} 0 0" />
         <geometry>
           <cylinder radius="0.15" length="0.05" />
@@ -46,7 +48,7 @@
       <inertial>
         <!-- <origin xyz="0 0 0" rpy="${pi/2} 0 0" /> -->
-        <origin xyz="0 0 0" rpy="0 0 0" />
-        <mass value="2" />
-        <xacro:cylinder_inertia m="2" r="0.15" h="0.05" />
+        <origin xyz="0 0 0" rpy="${pi/2} 0 0" />
+        <mass value="3" />
+        <xacro:cylinder_inertia m="3" r="0.15" h="0.05" />
       </inertial>
     </link>
@@ -54,6 +56,6 @@
       <parent link="base" />
       <child link="${side}_wheel_link" />
-      <origin xyz="${reflect_x * 0.25} ${reflect_y * 0.25} 0" rpy="1.570796 0 0" />
-      <axis xyz="0 0 -1" />
+      <origin xyz="${reflect_x * 0.25} ${reflect_y * 0.25} 0" />
+      <axis xyz="0 1 0" />
       <dynamics damping="0.8" friction="100.0" />
     </joint>
@@ -61,8 +63,8 @@
     <xacro:wheel_transmission prefix="${side}" />
   </xacro:macro>
-  <xacro:wheel side="left_front" reflect_x="-1" reflect_y="-1" />
-  <xacro:wheel side="left_back" reflect_x="1" reflect_y="-1" />
-  <xacro:wheel side="right_front" reflect_x="-1" reflect_y="1" />
-  <xacro:wheel side="right_back" reflect_x="1" reflect_y="1" />
+  <xacro:wheel side="left_front" reflect_x="1" reflect_y="1" />
+  <xacro:wheel side="left_back" reflect_x="-1" reflect_y="1" />
+  <xacro:wheel side="right_front" reflect_x="1" reflect_y="-1" />
+  <xacro:wheel side="right_back" reflect_x="-1" reflect_y="-1" />
   <link name="imu_link" />
   <joint name="imu_joint" type="fixed">
