Commit message: xacro works

File: tennis-description/urdf/leo.gazebo.xacro (robot description, xacro)
@@ -23,5 +23,5 @@
     </plugin>
   </gazebo>
-  <gazebo reference="base_link">
+  <gazebo reference="base">
     <material>Gazebo/Blue</material>
   </gazebo>

File: tennis-description/urdf/leo.xacro (robot description, xacro)
@@ -3,4 +3,10 @@
   <xacro:include filename="$(find tennis-description)/urdf/leo.gazebo.xacro" />
   <xacro:include filename="$(find tennis-description)/urdf/transmission.xacro" />
+  <xacro:property name="robotlxx" value="0.385" />
+  <xacro:property name="robotlxy" value="0" />
+  <xacro:property name="robotlxz" value="0" />
+  <xacro:property name="robotlyy" value="1.92098166" />
+  <xacro:property name="robotlyz" value="0" />
+  <xacro:property name="robotlzz" value="1.844169" />
   <link name="base">
     <visual>
@@ -16,5 +22,12 @@
       </geometry>
     </collision>
+    <inertial>
+      <mass value="36" />
+      <inertia ixx="${robotlxx}" ixy="${robotlxy}" ixz="${robotlxz}" iyy="${robotlyy}" iyz="${robotlyz}" izz="${robotlzz}" />
+    </inertial>
   </link>
+  <xacro:macro name="cylinder_inertia" params="m r h">
+    <inertia ixx="${m*(3*r*r+h*h)/12}" ixy="0" ixz="0" iyy="${m*(3*r*r+h*h)/12}" iyz="0" izz="${m*r*r/2}" />
+  </xacro:macro>
   <xacro:macro name="wheel" params="side reflect_x reflect_y">
     <link name="wheel_${side}">
@@ -31,5 +44,6 @@
       <inertial>
         <origin xyz="0 0 0" rpy="${pi/2} 0 0" />
-        <mass value="${wheelmass}" />
+        <mass value="1" />
+        <xacro:cylinder_inertia m="1" r="0.15" h="0.05" />
       </inertial>
     </link>
@@ -39,4 +53,5 @@
       <origin xyz="${reflect_x * 0.5} ${reflect_y * 0.5} 0" rpy="1.570796 0 0" />
       <axis xyz="0 0 1" />
+      <!-- <dynamics damping="0.8" friction="2.0" /> -->
     </joint>
   </xacro:macro>
@@ -47,7 +62,17 @@
   <link name="imu_link" />
   <joint name="imu_joint" type="fixed">
-    <parent link="base_link" />
+    <parent link="base" />
     <child link="imu_link" />
     <origin xyz="0.35 -0.1 0" rpy="0 0 0" />
+  </joint>
+  <!-- Create a root link with no inertia to make the solver happy and raise the robot above the floor -->
+  <link name="base_root">
+    <!-- <origin xyz="${bodyx} ${bodyy} ${bodyz}" rpy="${bodyroll} ${bodypitch} ${bodyyaw}" /> -->
+  </link>
+  <!-- Connect that link to the base link in the middle of the robot -->
+  <joint name="base_link_joint" type="fixed">
+    <origin xyz="0 0 0.15" rpy="0 0 0" />
+    <parent link="base_root" />
+    <child link="base" />
   </joint>
   <xacro:include filename="$(find gazebo_plugins)/test/multi_robot_scenario/xacro/laser/hokuyo.xacro" />

Commit message: works kinda

File: tennis-description/urdf/leo.gazebo.xacro (robot description, xacro)
@@ -2,13 +2,8 @@
 <robot xmlns:xacro="http://www.ros.org/wiki/xacro" name="leo">
   <gazebo>
-    <plugin name="gazebo_ros_control" filename="libgazebo_ros_control.so">
-      <robotNamespace>leo</robotNamespace>
-    </plugin>
-  </gazebo>
-  <gazebo>
     <plugin name="differential_drive_controller" filename="libgazebo_ros_diff_drive.so">
       <updateRate>100</updateRate>
-      <leftJoint>left_front</leftJoint>
-      <rightJoint>right_front</rightJoint>
+      <leftJoint>left_front_wheel_joint</leftJoint>
+      <rightJoint>right_front_wheel_joint</rightJoint>
       <wheelSeparation>0.33</wheelSeparation>
       <wheelDiameter>0.3</wheelDiameter>
@@ -19,6 +14,6 @@
       <odometryFrame>odom</odometryFrame>
       <robotBaseFrame>base_root</robotBaseFrame>
-      <!-- <odometrySource>1</odometrySource> -->
-      <publishWheelTF>true</publishWheelTF>
+      <odometrySource>1</odometrySource>
+      <publishWheelTF>false</publishWheelTF>
       <publishOdomTF>true</publishOdomTF>
       <publishWheelJointState>true</publishWheelJointState>
@@ -55,3 +50,8 @@
     </gazebo>
   </xacro:macro>
+  <gazebo>
+    <plugin name="gazebo_ros_control" filename="libgazebo_ros_control.so">
+      <robotNamespace>leo</robotNamespace>
+    </plugin>
+  </gazebo>
 </robot>

File: tennis-description/urdf/leo.xacro (robot description, xacro)
@@ -31,5 +31,5 @@
   </xacro:macro>
   <xacro:macro name="wheel" params="side reflect_x reflect_y">
-    <link name="wheel_${side}">
+    <link name="${side}_wheel_link">
       <visual>
         <geometry>
@@ -48,7 +48,7 @@
       </inertial>
     </link>
-    <joint name="base_wheel_${side}_joint" type="continuous">
+    <joint name="${side}_wheel_joint" type="continuous">
       <parent link="base" />
-      <child link="wheel_${side}" />
+      <child link="${side}_wheel_link" />
       <origin xyz="${reflect_x * 0.25} ${reflect_y * 0.25} 0" rpy="1.570796 0 0" />
       <axis xyz="0 0 1" />
@@ -68,4 +68,10 @@
     <origin xyz="0.35 -0.1 0" rpy="0 0 0" />
   </joint>
+  <link name="odom" />
+  <joint name="odom_joint" type="fixed">
+    <parent link="base" />
+    <child link="odom" />
+    <origin xyz="0 0 0 " rpy="0 0 0" />
+  </joint>
   <!-- Create a root link with no inertia to make the solver happy and raise the robot above the floor -->
   <link name="base_root">
@@ -80,4 +86,4 @@
   <!-- <xacro:include filename="$(find gazebo_plugins)/test/multi_robot_scenario/xacro/laser/hokuyo.xacro" /> -->
   <xacro:include filename="$(find tennis-description)/urdf/laser.xacro" />
-  <xacro:laser name="laser_vert_bottom" parent="base" xyz="0.3157984464801903 -0.002068548615034871 0.25" rpy="3.14159 0.0 0.0" meshes="$(find tennis-description)/meshes" />
+  <xacro:laser name="laser_vert_bottom" parent="base" xyz="0.3157984464801903 -0.002068548615034871 0.25" rpy="3.14159 0.0 0.0" meshes="$(find tennis-description)/meshes/laser" />
 </robot>

Commit message: added xacro files for camera and lidar, removed old files

File: tennis-description/urdf/leo.gazebo.xacro (robot description, xacro)
@@ -30,5 +30,5 @@
       <always_on>true</always_on>
       <update_rate>30</update_rate>
-      <visualize>false</visualize>
+      <visualize>true</visualize>
       <topic>imu</topic>
       <plugin filename="libgazebo_ros_imu_sensor.so" name="imu_plugin">
@@ -48,7 +48,10 @@
   <xacro:macro name="wheel_gazebo" params="prefix">
     <gazebo reference="${prefix}_wheel_link">
-      <material>Gazebo/Grey</material>
-      <mu1 value="0.6" />
-      <mu2 value="0.6" />
+      <material>Gazebo/DarkGrey</material>
+      <mu1 value="0.9" />
+      <mu2 value="0.9" />
+      <selfCollide>false</selfCollide>
+      <!-- <kp value="10000000.0" /> -->
+      <!-- <kd value="1" /> -->
     </gazebo>
   </xacro:macro>

File: tennis-description/urdf/leo.xacro (robot description, xacro)
@@ -3,4 +3,6 @@
   <xacro:include filename="$(find tennis-description)/urdf/leo.gazebo.xacro" />
   <xacro:include filename="$(find tennis-description)/urdf/transmission.xacro" />
+  <xacro:include filename="$(find tennis-description)/urdf/camera.xacro" />
+  <xacro:include filename="$(find tennis-description)/urdf/rplidar.xacro" />
   <xacro:property name="robotlxx" value="0.385" />
   <xacro:property name="robotlxy" value="0" />
@@ -49,13 +51,4 @@
       </inertial>
     </link>
-    <gazebo reference="${side}_wheel_link">
-      <!-- <material>Gazebo/DarkGrey</mate10ial> -->
-      <selfCollide>false</selfCollide>
-      <!-- <mu value="0.9" /> -->
-      <!-- <mu2 value="0.9" /> -->
-      <kp value="10000000.0" />
-      <kd value="1" />
-      <!-- <fdir1 value="1 0 0" /> -->
-    </gazebo>
     <joint name="${side}_wheel_joint" type="continuous">
       <parent link="base" />
@@ -76,5 +69,5 @@
     <parent link="base" />
     <child link="imu_link" />
-    <origin xyz="0.35 -0.1 0" rpy="0 0 0" />
+    <origin xyz="0.0 0.0 0" rpy="0 0 0" />
   </joint>
   <link name="odom" />
@@ -88,5 +81,5 @@
     <!-- <origin xyz="${bodyx} ${bodyy} ${bodyz}" rpy="${bodyroll} ${bodypitch} ${bodyyaw}" /> -->
   </link>
-  <!-- Connect that link to the base link in the middle of the robot -->
+  <!-- Connect that link to the base link in middle of the robot -->
   <joint name="base_root_joint" type="fixed">
     <origin xyz="0 0 0.15" rpy="0 0 0" />
@@ -94,6 +87,12 @@
     <child link="base" />
   </joint>
+  <!-- camera definitions -->
+  <xacro:camera name="front_camera" parent="base" xyz="0.5 0 0.2" rpy="0 0 0" />
+  <xacro:camera name="rear_camera" parent="base" xyz="-0.5 0 0.2" rpy="0 0 ${pi}" />
+  <!-- lidar definition -->
+  <xacro:rplidar name="lidar" parent="base" xyz="0 0 0.25" rpy="0 0 0" />
+  <!-- old lidar stuff -->
   <!-- <xacro:include filename="$(find gazebo_plugins)/test/multi_robot_scenario/xacro/laser/hokuyo.xacro" /> -->
-  <xacro:include filename="$(find tennis-description)/urdf/laser.xacro" />
-  <xacro:laser name="laser_vert_bottom" parent="base" xyz="0.3157984464801903 -0.002068548615034871 0.25" rpy="3.14159 0.0 0.0" meshes="$(find tennis-description)/meshes/laser" />
+  <!-- <xacro:include filename="$(find tennis-description)/urdf/laser.xacro" /> -->
+  <!-- <xacro:laser name="lidar" parent="base" xyz="0.3157984464801903 -0.002068548615034871 0.25" rpy="3.14159 0.0 0.0" meshes="$(find tennis-description)/meshes/laser" /> -->
 </robot>

Commit message: tennis balls are now yellow. Added a node to spawn the balls

File: tennis-description/urdf/leo.gazebo.xacro (robot description, xacro)
@@ -1,25 +1,4 @@
 <?xml version="1.0"?>
 <robot xmlns:xacro="http://www.ros.org/wiki/xacro" name="leo">
-  <!-- <gazebo> -->
-  <!--   <plugin name="skid_steer" filename="libgazebo_ros_skid_steer_drive.so"> -->
-  <!--     <updateRate>100</updateRate> -->
-  <!--     <leftFrontJoint>left_front_wheel_joint</leftFrontJoint> -->
-  <!--     <leftRearJoint>left_back_wheel_joint</leftRearJoint> -->
-  <!--     <rightFrontJoint>right_front_wheel_joint</rightFrontJoint> -->
-  <!--     <rightRearJoint>right_back_wheel_joint</rightRearJoint> -->
-  <!--     <wheelSeparation>0.33</wheelSeparation> -->
-  <!--     <wheelDiameter>0.3</wheelDiameter> -->
-  <!--     <wheelAcceleration>false</wheelAcceleration> -->
-  <!--     <torque>100</torque> -->
-  <!--     <commandTopic>diff/cmd_vel</commandTopic> -->
-  <!--     <odometryTopic>diff/odom</odometryTopic> -->
-  <!--     <odometryFrame>odom</odometryFrame> -->
-  <!--     <robotBaseFrame>base_root</robotBaseFrame> -->
-  <!--     <odometrySource>1</odometrySource> -->
-  <!--     <publishWheelTF>false</publishWheelTF> -->
-  <!--     <publishOdomTF>true</publishOdomTF> -->
-  <!--     <publishWheelJointState>true</publishWheelJointState> -->
-  <!--   </plugin> -->
-  <!-- </gazebo> -->
   <gazebo reference="base">
     <material>Gazebo/Blue</material>
@@ -46,4 +25,26 @@
     </sensor>
   </gazebo>
+  <gazebo reference="vacuum_link">
+    <material>Gazebo/Red</material>
+    <sensor name="vacuum_bumper" type="contact">
+      <selfCollide>false</selfCollide>
+      <alwaysOn>true</alwaysOn>
+      <updateRate>20.0</updateRate>
+      <!-- <contact> -->
+      <!-- find with gz sdf -p leo.xacro -->
+      <!--   <collision>leo/base_root_fixed_joint_lump__vacuum_link_collision_collision_4</collision> -->
+      <!-- </contact> -->
+      <contact>
+        <collision name="bump_sensor_collision_collision"></collision>
+      </contact>
+      <plugin name="gazebo_ros_bumper_controller" filename="libgazebo_ros_bumper.so">
+        <robotNamespace>leo</robotNamespace>
+        <bumperTopicName>vacuum_contacts</bumperTopicName>
+        <frameName>world</frameName>
+        <alwaysOn>true</alwaysOn>
+        <updateRate>20.0</updateRate>
+      </plugin>
+    </sensor>
+  </gazebo>
   <xacro:macro name="wheel_gazebo" params="prefix">
     <gazebo reference="${prefix}_wheel_link">

File: tennis-description/urdf/leo.xacro (robot description, xacro)
@@ -73,10 +73,21 @@
     <origin xyz="0.0 0.0 0" rpy="0 0 0" />
   </joint>
-  <!-- <link name="odom" /> -->
-  <!-- <joint name="odom_joint" type="fixed"> -->
-  <!--   <parent link="odom" /> -->
-  <!--   <child link="base_root" /> -->
-  <!--   <origin xyz="0 0 0 " rpy="0 0 0" /> -->
-  <!-- </joint> -->
+  <link name="vacuum_link">
+    <visual>
+      <geometry>
+        <box size="0.01 0.33 0.1" />
+      </geometry>
+    </visual>
+    <collision>
+      <geometry>
+        <box size="0.01 0.33 0.1" />
+      </geometry>
+    </collision>
+  </link>
+  <joint name="vacuum_joint" type="fixed">
+    <origin xyz="0.52 0 -0.10" />
+    <parent link="base" />
+    <child link="vacuum_link" />
+  </joint>
   <!-- Create a root link with no inertia to make the solver happy and raise the robot above the floor -->
   <link name="base_root">

Commit message: bumper plugin works

File: tennis-description/urdf/leo.gazebo.xacro (robot description, xacro)
@@ -36,5 +36,5 @@
       <!-- </contact> -->
       <contact>
-        <collision name="bump_sensor_collision_collision"></collision>
+        <collision>base_root_fixed_joint_lump__vacuum_link_collision_4</collision>
       </contact>
       <plugin name="gazebo_ros_bumper_controller" filename="libgazebo_ros_bumper.so">

File: tennis-description/urdf/leo.xacro (robot description, xacro)
@@ -86,5 +86,5 @@
   </link>
   <joint name="vacuum_joint" type="fixed">
-    <origin xyz="0.52 0 -0.10" />
+    <origin xyz="0.52 0 -0.07" />
     <parent link="base" />
     <child link="vacuum_link" />
